Commit message: Completes (minimal) URDF setup
Can now launch and control the robot model. Setup just like normal, just without connecting to the arduino. This can be used to simulate what the robot will do with certain input, and serves as a stepping stone to proper SLAM

File: rossystem/src/acr_setup/config/acr.urdf (robot description, URDF)
Before this commit: robot ACR, 1 links, 0 joints
Links:
- added link lidar_link; visual box size=.1 .1 .1
- link base_link: geometry visual box size=1 .7 .2
Joints:
- added joint my_joint: type fixed, parent base_link, child lidar_link, origin xyz=.45 0 .15
