Commit message: Adds a global launch file
You can now launch the robot simulation from the acr_setup node. The rosserial node is not yet included, simply because I haven't experimented enough with it yet. Was a bit too exited that the mapping was finally working

File: ros/src/acr_setup/config/acr.urdf (robot description, URDF)
Before this commit: robot ACR, 2 links, 1 joints
Links:
- removed link lidar_link
- added link base_scan; visual box size=.1 .1 .1
Joints:
- joint my_joint: child lidar_link -> base_scan

Commit message: Adds acr model to urdf
Fixes leddar configuration to work with gmapping

Lidar didn't work properly after the 'big refactor', so decided to do it from scratch. Found some issues in the process including a static tf transform, which rotated and translated the lidar, which made it incompatible with the gmapping node.

Adds serial node and ACR models to setup

Serial node is now also started in the launch file. The default port is /dev/ttyACM0 and can only be changed by modifying the launch file itself, there should be a paramater made for the arduino and leddar ports. In addition to that, there is now an actual model of the robot riding around in the simulation. Unofficial name got updated to Jimmy.

Removes weird artifact

File with the name '--' popped up, no clue how, but deleted it.

Removes redundant files and renaming

Revert "Removes weird artifact"

This reverts commit a0cf9eaabd7a517052cd73b5b5680829e711d7cc.

:q

Removes weird artifact

File with the name '--' popped up, no clue how, but deleted it.

Revert "Removes redundant files and renaming"

This reverts commit b132091cd5773be8b0a341976c631b1c0ce4e858.

:q

Removes devel from repo

Removes redundant 3d files

Removes redundant 3d files

Adds gitlarge file support

File: ros/src/acr_setup/config/acr.urdf (robot description, URDF)
Before this commit: robot ACR, 2 links, 1 joints
Links:
- link base_link: geometry visual mesh filename=package://acr_setup/config/ACR.stl

Commit message: Final commit to project

File: ros/src/acr_setup/config/acr.urdf (robot description, URDF)
Before this commit: robot ACR, 2 links, 1 joints
Joints:
- joint my_joint: origin xyz=.45 0 .15 -> xyz=.45 0 .15 rpy=180 0 0 
